Commit message: Control Loop and Visualization

File: 6dof_description.urdf (robot description, URDF)
Before this commit: robot 6dof_robot, 7 links, 6 joints
Links:
- link base_link: geometry visual cylinder length=0.05 radius=0.03
- link link1: geometry visual cylinder length=0.014 radius=0.03
- link link2: geometry visual cylinder length=0.105 radius=0.03
- link link3: geometry visual cylinder length=0.05 radius=0.03
- link link4: geometry visual cylinder length=0.065 radius=0.03
- link link5: geometry visual cylinder length=0.06 radius=0.03
- link link6: geometry visual cylinder length=0.05 radius=0.03
Joints:
- joint gripper: origin xyz=0 0.084 0 rpy=1.57 0 0 -> xyz=0 0.06 0 rpy=1.57 0 0
- joint joint1: origin xyz=0 0 0.12 rpy=-1.57 0 0 -> xyz=0 0 0.014 rpy=-1.57 0 0
- joint joint2: origin xyz=0 -0.225 0 rpy=0 0 -1.57 -> xyz=0 -0.105 0 rpy=0 0 -1.57
- joint joint3: origin xyz=0 0 0.052 rpy=1.57 0 0 -> xyz=0 0.05 0  rpy=1.57 0 0
- joint joint4: origin xyz=0 0 -0.09 rpy=-1.57 0 0 -> xyz=0 0 -0.065 rpy=-1.57 0 0
- joint rotary_base: origin xyz=0 0 0.02 rpy=0 0 0 -> xyz=0 0 0.05 rpy=0 0 0

Commit message: Added feature work

File: 6dof_description.urdf (robot description, URDF)
Before this commit: robot 6dof_robot, 7 links, 6 joints
Joints:
- joint gripper: origin xyz=0 0.06 0 rpy=1.57 0 0 -> xyz=0 -0.06 0 rpy=-1.57 0 0
- joint joint1: origin xyz=0 0 0.014 rpy=-1.57 0 0 -> xyz=0 0 0.014 rpy=1.57 0 0
- joint joint2: origin xyz=0 -0.105 0 rpy=0 0 -1.57 -> xyz=0 0.105 0 rpy=0 0 1.57
- joint joint3: origin xyz=0 0.05 0  rpy=1.57 0 0 -> xyz=0 -0.05 0  rpy=-1.57 0 0
- joint joint4: origin xyz=0 0 -0.065 rpy=-1.57 0 0 -> xyz=0 0 -0.065 rpy=1.57 0 0

Commit message: actual position implementation

File: 6dof_description.urdf (robot description, URDF)
Before this commit: robot 6dof_robot, 7 links, 6 joints
Links:
- link base_link: geometry visual cylinder length=0.055 radius=0.01
- link link1: geometry visual cylinder length=0.02 radius=0.01
- link link2: geometry visual cylinder length=0.105 radius=0.01
- link link3: geometry visual cylinder length=0.055 radius=0.01
- link link4: geometry visual cylinder length=0.065 radius=0.01
- link link5: geometry visual cylinder length=0.06 radius=0.01
- link link6: geometry visual cylinder length=0.04 radius=0.01
Joints:
- joint joint1: origin xyz=0 0 0.014 rpy=1.57 0 0 -> xyz=0 0 0.02 rpy=1.57 0 0
- joint joint3: origin xyz=0 -0.05 0  rpy=-1.57 0 0 -> xyz=0 -0.055 0  rpy=-1.57 0 0
- joint rotary_base: origin xyz=0 0 0.05 rpy=0 0 0 -> xyz=0 0 0.055 rpy=0 0 0

Commit message: added circular trajectory

File: 6dof_description.urdf (robot description, URDF)
Before this commit: robot 6dof_robot, 7 links, 6 joints
Links:
- link link1: geometry visual cylinder length=0.013 radius=0.01
- link link3: geometry visual cylinder length=0.045 radius=0.01
- link link4: geometry visual cylinder length=0.053 radius=0.01
- link link5: geometry visual cylinder length=0.053 radius=0.01
- link link6: geometry visual cylinder length=0.045 radius=0.01
Joints:
- joint gripper: origin xyz=0 -0.06 0 rpy=-1.57 0 0 -> xyz=0 -0.053 0 rpy=-1.57 0 0
- joint joint1: origin xyz=0 0 0.02 rpy=1.57 0 0 -> xyz=0 0 0.013 rpy=1.57 0 0
- joint joint3: origin xyz=0 -0.055 0  rpy=-1.57 0 0 -> xyz=0 -0.045 0  rpy=-1.57 0 0
- joint joint4: origin xyz=0 0 -0.065 rpy=1.57 0 0 -> xyz=0 0 -0.053 rpy=1.57 0 0

Commit message: Started Report

File: 6dof_description.urdf (robot description, URDF)
Before this commit: robot 6dof_robot, 7 links, 6 joints
Links:
- link base_link: geometry collision cylinder length=0.055 radius=0.01; visual cylinder length=0.055 radius=0.01
- link link1: geometry collision cylinder length=0.013 radius=0.01; visual cylinder length=0.013 radius=0.01
- link link2: geometry collision cylinder length=0.105 radius=0.01; visual cylinder length=0.105 radius=0.01
- link link3: geometry visual cylinder length=0.047 radius=0.01
- link link4: geometry collision cylinder length=0.086 radius=0.01; visual cylinder length=0.086 radius=0.01
- link link5: geometry collision cylinder length=0.051 radius=0.01; visual cylinder length=0.051 radius=0.01
- link link6: geometry collision cylinder length=0.047 radius=0.01; visual cylinder length=0.047 radius=0.01
Joints:
- joint gripper: origin xyz=0 -0.053 0 rpy=-1.57 0 0 -> xyz=0 -0.051 0 rpy=-1.57 0 0
- joint joint3: origin xyz=0 -0.045 0  rpy=-1.57 0 0 -> xyz=0 -0.047 0  rpy=-1.57 0 0
- joint joint4: origin xyz=0 0 -0.053 rpy=1.57 0 0 -> xyz=0 0 -0.086 rpy=1.57 0 0
